File: cell/electronics/pcb.sch (EAGLE design)
At the start: 27 parts, among them IC2 L293D, M1 M02PTH3, M2 M02PTH3, Q1 MOSFET-NCHANNEL2N7000, Q2 MOSFET-NCHANNEL2N7000, SW1 M02PTH3, SW2 M02PTH3, SW3 M02PTH3, SW4 M02PTH3, SW5 M02PTH3

Commit message: Relaying out the board
laying out the board again for production, easier to read, components
aligned and placed better. ready for first rev production
Parts:
- added JP9: (no value), SparkFun-Connectors:M03LONGPADS
- renumbered IC2 to L293D, JP2 to LED1, JP3 to LED2, JP4 to SW0, JP5 to SV2, JP6 to SV1, U$1 to ATTINY
Connections:
- new net N$17: JP9.2, L293D.VCC2
- net 5V: now also JP9.1, R1.2; no longer R3.2
- net GND: now also JP8.1, R3.1; no longer JP8.3, R1.1
- net N$10: now also R1.1; no longer R3.1
- net N$12: now also R2.2; no longer R1.2
- net N$13: now also R3.2; no longer R2.2
- net VCC: now also JP8.3, JP9.3; no longer JP8.1, L293D.VCC2
Other:
- moved on the sheet: R1, R2, R3
